File: Ears.kicad_pcb (KiCad board)
At the start: 2 copper layers, 113.8 x 147 mm, 197 parts, among them J1 Conn_01x06_Male

Commit message: Fixed fill region not assigned to the proper net.
Signed-off-by: Aaron Williams <aaron.w2@gmail.com>
Routing:
- removed copper zone on B.Cu, net (none)
Changed lines of the file:
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@@
     )
   )
-  (zone (net 0) (net_name "") (layer B.Cu) (hatch edge 0.508)
+  (zone (net 1) (net_name VCC) (layer B.Cu) (hatch edge 0.508)
     (priority 2)
     (connect_pads yes (clearance 0.508))

Commit message: Fixed fill area and added back silkscreen
Signed-off-by: Aaron Williams <aaron.w2@gmail.com>
Other:
- board text added: "Flex Ear LEDs Copyright © 2019 by Aaron Williams Revision 1.0.2"
Changed lines of the file:
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@@
   (general
     (thickness 1.6)
-    (drawings 102)
+    (drawings 103)
     (tracks 1882)
     (zones 0)
@@
   )
   (setup
-    (last_trace_width 0.8)
+    (last_trace_width 0.3)
     (user_trace_width 0.3)
     (user_trace_width 0.5)
@@
     )
   )
+  (gr_text "Flex Ear LEDs Copyright © 2019 by Aaron Williams\nRevision 1.0.2" (at 73.3 127.1) (layer B.SilkS)
+    (effects (font (size 1.5 1.5) (thickness 0.3)) (justify mirror))
+  )
   (gr_line (start 66 162.4) (end 66 159.7) (layer Cmts.User) (width 0.15))
